File: ControllerSchematicKiCAD/ConttrollerSchematic/ConttrollerSchematic.kicad_sch (KiCad schematic)
At the start: 9 parts, among them J1 Conn_01x06, J2 Conn_01x15_Pin, J3 Conn_01x15_Pin, SW1 SW_Push, SW2 SW_Push

Commit message: Schematic updates
lots of stuff
Parts:
- removed D1, D2: LED, LED_THT:LED_D5.0mm, symbol Device:LED
- removed J1: Conn_01x06, Connector_PinSocket_2.54mm:PinSocket_1x06_P2.54mm_Horizontal, symbol Connector_Generic:Conn_01x06
- removed J2, J3: Conn_01x15_Pin, Connector_PinHeader_1.00mm:PinHeader_1x15_P1.00mm_Vertical, symbol Connector:Conn_01x15_Pin
- added Joystick1: Conn_01x05_Socket, Connector_PinSocket_2.54mm:PinSocket_1x05_P2.54mm_Horizontal, symbol Connector:Conn_01x05_Socket
- added LeftESP1, RightESP1: Conn_01x15_Pin, Connector_PinSocket_2.54mm:PinSocket_1x15_P2.54mm_Vertical, symbol Connector:Conn_01x15_Pin
- added Screen1: Conn_01x04_Socket, Connector_PinSocket_1.00mm:PinSocket_1x04_P1.00mm_Vertical, symbol Connector:Conn_01x04_Socket
- renumbered SW1 to Button1, SW2 to Button2, D3 to LED1, D4 to LED2
Connections:
- net GND: now reaches Button2.1
- net GND: now also Button1.1, LED1.1 (K), LED2.1 (K), Joystick1.5 (Ground), LeftESP1.2 (Pin_2), RightESP1.1 (Pin_1), Screen1.4 (Ground)
- net L3: now reaches Button1.2
- net L3: now also LeftESP1.3 (Pin_3); no longer Button2.2
- net L10: now reaches LED1.2 (A)
- net L10: now also LeftESP1.10 (Pin_10)
- net L9: now reaches LED2.2 (A)
- net L9: now also LeftESP1.9 (Pin_9)
- new net L5: Joystick1.1 (Button), LeftESP1.5 (Pin_5)
- new net L6: Button2.2, LeftESP1.6 (Pin_6)
- new net L7: Joystick1.3 (X-position), LeftESP1.7 (Pin_7)
- new net L8: Joystick1.2 (Y-position), LeftESP1.8 (Pin_8)
- new net R11: RightESP1.14 (Pin_14), Screen1.2 (SCL)
- new net R14: RightESP1.11 (Pin_11), Screen1.1 (SDA)
- new net V+: Joystick1.4 (+V), RightESP1.2 (Pin_2), Screen1.3 (VCC)
- no-connect marks 0 -> 18
Other:
- moved on the sheet: Button1, Button2, LED1, LED2

Commit message: auto routed
heheh
Parts:
- renumbered Button1 to Button12222
Changed lines of the file:
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@@
 	(global_label "GND"
 		(shape input)
+		(at 220.98 71.12 180)
+		(fields_autoplaced yes)
+		(effects
+			(font
+				(size 1.27 1.27)
+			)
+			(justify right)
+		)
+		(property "Intersheetrefs" "${INTERSHEET_REFS}"
+			(at 214.1243 71.12 0)
+			(effects
+				(font
+					(size 1.27 1.27)
+				)
+				(justify right)
+				(hide yes)
+			)
+		)
+	)
+	(global_label "GND"
+		(shape input)
+		(at 64.77 90.17 180)
+		(fields_autoplaced yes)
+		(effects
+			(font
+				(size 1.27 1.27)
+			)
+			(justify right)
+		)
+		(property "Intersheetrefs" "${INTERSHEET_REFS}"
+			(at 57.9143 90.17 0)
+			(effects
+				(font
+					(size 1.27 1.27)
+				)
+				(justify right)
+				(hide yes)
+			)
+		)
+	)
+	(global_label "GND"
+		(shape input)
+		(at 143.51 92.71 180)
+		(fields_autoplaced yes)
+		(effects
+			(font
+				(size 1.27 1.27)
+			)
+			(justify right)
+		)
+		(property "Intersheetrefs" "${INTERSHEET_REFS}"
+			(at 136.6543 92.71 0)
+			(effects
+				(font
+					(size 1.27 1.27)
+				)
+				(justify right)
+				(hide yes)
+			)
+		)
+	)
+	(global_label "GND"
+		(shape input)
+		(at 105.41 77.47 180)
+		(fields_autoplaced yes)
+		(effects
+			(font
+				(size 1.27 1.27)
+			)
+			(justify right)
+		)
+		(property "Intersheetrefs" "${INTERSHEET_REFS}"
+			(at 98.5543 77.47 0)
+			(effects
+				(font
+					(size 1.27 1.27)
+				)
+				(justify right)
+				(hide yes)
+			)
+		)
+	)
+	(global_label "V+"
+		(shape input)
+		(at 205.74 92.71 0)
+		(fields_autoplaced yes)
+		(effects
+			(font
+				(size 1.27 1.27)
+			)
+			(justify left)
+		)
+		(property "Intersheetrefs" "${INTERSHEET_REFS}"
+			(at 211.3862 92.71 0)
+			(effects
+				(font
+					(size 1.27 1.27)
+				)
+				(justify left)
+				(hide yes)
+			)
+		)
+	)
+	(global_label "GND"
+		(shape input)
 		(at 64.77 73.66 180)
 		(fields_autoplaced yes)
@@
 				)
 				(justify right)
-				(hide yes)
-			)
-		)
-	)
-	(global_label "GND"
-		(shape input)
-		(at 220.98 71.12 180)
-		(fields_autoplaced yes)
-		(effects
-			(font
-				(size 1.27 1.27)
-			)
-			(justify right)
-		)
-		(property "Intersheetrefs" "${INTERSHEET_REFS}"
-			(at 214.1243 71.12 0)
-			(effects
-				(font
-					(size 1.27 1.27)
-				)
-				(justify right)
-				(hide yes)
-			)
-		)
-	)
-	(global_label "GND"
-		(shape input)
-		(at 64.77 90.17 180)
-		(fields_autoplaced yes)
-		(effects
-			(font
-				(size 1.27 1.27)
-			)
-			(justify right)
-		)
-		(property "Intersheetrefs" "${INTERSHEET_REFS}"
-			(at 57.9143 90.17 0)
-			(effects
-				(font
-					(size 1.27 1.27)
-				)
-				(justify right)
-				(hide yes)
-			)
-		)
-	)
-	(global_label "GND"
-		(shape input)
-		(at 143.51 92.71 180)
-		(fields_autoplaced yes)
-		(effects
-			(font
-				(size 1.27 1.27)
-			)
-			(justify right)
-		)
-		(property "Intersheetrefs" "${INTERSHEET_REFS}"
-			(at 136.6543 92.71 0)
-			(effects
-				(font
-					(size 1.27 1.27)
-				)
-				(justify right)
-				(hide yes)
-			)
-		)
-	)
-	(global_label "GND"
-		(shape input)
-		(at 105.41 77.47 180)
-		(fields_autoplaced yes)
-		(effects
-			(font
-				(size 1.27 1.27)
-			)
-			(justify right)
-		)
-		(property "Intersheetrefs" "${INTERSHEET_REFS}"
-			(at 98.5543 77.47 0)
-			(effects
-				(font
-					(size 1.27 1.27)
-				)
-				(justify right)
-				(hide yes)
-			)
-		)
-	)
-	(global_label "V+"
-		(shape input)
-		(at 205.74 92.71 0)
-		(fields_autoplaced yes)
-		(effects
-			(font
-				(size 1.27 1.27)
-			)
-			(justify left)
-		)
-		(property "Intersheetrefs" "${INTERSHEET_REFS}"
-			(at 211.3862 92.71 0)
-			(effects
-				(font
-					(size 1.27 1.27)
-				)
-				(justify left)
 				(hide yes)
 			)
@@
 		(dnp no)
 		(fields_autoplaced yes)
-		(property "Reference" "Button1"
+		(property "Reference" "Button12222"
 			(at 73.66 66.04 0)
 			(effects
@@
 			(project ""
 				(path "/078b711c-5737-48ab-b356-b914bbaeec72"
-					(reference "Button1")
+					(reference "Button12222")
 					(unit 1)
 				)
