File: RobotSchematicKICAD/RobotSchematicPCB/RobotSchematicPCB.kicad_sch (KiCad schematic)
At the start: 0 parts

Commit message: imported from 3d model for exact dimensions
I imported the dxf from the model for the controller and then I made that the edge cuts for the board. I also added some art
Parts:
- added BOOTPULL1, ENPULL1, R1: 10k, Resistor_SMD:R_0603_1608Metric, symbol Device:R
- added C1, C2: 10u, Capacitor_SMD:C_0603_1608Metric, symbol Device:C_US
- added D1, D2, D3, D4, D5, D6, D7, D8: LED, LED_THT:LED_D3.0mm, symbol Device:LED
- added LDO1: AMS1117-3.3, Resistor_SMD:R_0201_0603Metric, symbol Regulator_Linear:AMS1117-3.3
- added LEDR1, LEDR2, LEDR3, LEDR4, LEDR5, LEDR6, LEDR7, LEDR8: 330, Resistor_SMD:R_0603_1608Metric, symbol Device:R_Small
- added SERVO1, SERVO10, SERVO11, SERVO12, SERVO2, SERVO3, SERVO4, SERVO5, SERVO6, SERVO7, SERVO8, SERVO9: Conn_01x03_Pin, Connector_Harwin:Harwin_M20-89003xx_1x03_P2.54mm_Horizontal, symbol Connector:Conn_01x03_Pin
- added SWBOOT1, SWEN1: SW_Push, Button_Switch_THT:SW_PUSH_6mm, symbol Switch:SW_Push
- added U1: PCA9685PW, Package_SO:TSSOP-28_4.4x9.7mm_P0.65mm, symbol Driver_LED:PCA9685PW
- added U2: ESP32-WROOM-32E, RF_Module:ESP32-WROOM-32D, symbol RF_Module:ESP32-WROOM-32E
- added U3: 74HC595, Package_SO:SOIC-16_3.9x9.9mm_P1.27mm, symbol 74xx:74HC595
- added U4: ESP32-C6-MINI-1, RF_Module:ESP32-C6-MINI-1, symbol RF_Module:ESP32-C6-MINI-1
- added XT90BATTERY1: Screw_Terminal_01x02, Connector_Phoenix_GMSTB:PhoenixContact_GMSTB_2,5_2-GF-7,62_1x02_P7.62mm_Horizontal_ThreadedFlange_MountHole, symbol Connector:Screw_Terminal_01x02
Connections:
- new net: D2.2 (A), LEDR2.2
- new net: D7.2 (A), LEDR7.2
- new net: C1.1, LDO1.3 (VI), XT90BATTERY1.1 (Pin_1)
- new net: ENPULL1.2, SWEN1.2, U2.3 (EN)
- new net: D5.2 (A), LEDR5.2
- new net: D4.2 (A), LEDR4.2
- new net: D6.2 (A), LEDR6.2
- new net: BOOTPULL1.2, SWBOOT1.2, U2.25 (IO0)
- new net: D8.2 (A), LEDR8.2
- new net: D1.2 (A), LEDR1.2
- new net: D3.2 (A), LEDR3.2
- new net: U4.1 (GND), U4.11 (GND), U4.14 (GND), U4.2 (GND), U4.36 (GND), U4.37 (GND), U4.38 (GND), U4.39 (GND), U4.40 (GND), U4.41 (GND), U4.42 (GND), U4.43 (GND), U4.44 (GND), U4.45 (GND), U4.46 (GND), U4.47 (GND), U4.48 (GND), U4.49 (GND), U4.50 (GND), U4.51 (GND), U4.52 (GND), U4.53 (GND)
- new net: R1.2, U1.23 (~{OE})
- new net 3V3: BOOTPULL1.1, C2.1, ENPULL1.1, LDO1.2 (VO), U1.28 (VDD), U2.2 (VDD), U3.10 (~{SRCLR}), U3.16 (VCC)
- new net 5V: SERVO1.3 (Pin_3), SERVO10.3 (Pin_3), SERVO11.3 (Pin_3), SERVO12.3 (Pin_3), SERVO2.3 (Pin_3), SERVO3.3 (Pin_3), SERVO4.3 (Pin_3), SERVO5.3 (Pin_3), SERVO6.3 (Pin_3), SERVO7.3 (Pin_3), SERVO8.3 (Pin_3), SERVO9.3 (Pin_3), U1.14 (VSS)
- new net GND: C1.2, C2.2, D1.1 (K), D2.1 (K), D3.1 (K), D4.1 (K), D5.1 (K), D6.1 (K), D7.1 (K), D8.1 (K), LDO1.1 (GND), R1.1, SERVO1.2 (Pin_2), SERVO10.2 (Pin_2), SERVO11.2 (Pin_2), SERVO12.2 (Pin_2), SERVO2.2 (Pin_2), SERVO3.2 (Pin_2), SERVO4.2 (Pin_2), SERVO5.2 (Pin_2), SERVO6.2 (Pin_2), SERVO7.2 (Pin_2), SERVO8.2 (Pin_2), SERVO9.2 (Pin_2), SWBOOT1.1, SWEN1.1, U1.1 (A0), U1.2 (A1), U1.24 (A5), U1.3 (A2), U1.4 (A3), U1.5 (A4), U2.1 (GND), U2.15 (GND), U2.38 (GND), U2.39 (GND), U3.13 (~{OE}), U3.8 (GND), XT90BATTERY1.2 (Pin_2)
- new net LED0: SERVO1.1 (Pin_1)
- new net LED1: SERVO2.1 (Pin_1), U1.6 (LED0), U3.15 (QA)
- new net LED10: SERVO11.1 (Pin_1), U1.15 (LED8)
- new net LED11: SERVO12.1 (Pin_1), U1.16 (LED9)
- new net LED12: U1.17 (LED10), U1.18 (LED11)
- new net LED2: SERVO3.1 (Pin_1), U3.1 (QB)
- new net LED3: SERVO4.1 (Pin_1), U1.7 (LED1), U3.2 (QC)
- new net LED4: SERVO5.1 (Pin_1), U1.8 (LED2), U3.3 (QD)
- new net LED5: SERVO6.1 (Pin_1), U1.9 (LED3), U3.4 (QE)
- new net LED6: SERVO7.1 (Pin_1), U1.10 (LED4), U3.5 (QF)
- new net LED7: SERVO8.1 (Pin_1), U1.11 (LED5), U3.6 (QG)
- new net LED8: SERVO9.1 (Pin_1), U1.12 (LED6), U3.7 (QH)
- new net LED9: SERVO10.1 (Pin_1), U1.13 (LED7)
- new net SCL: U1.26 (SCL), U2.36 (IO22)
- new net SDA: U1.27 (SDA), U2.33 (IO21)
- new net SR_CLK: U2.13 (IO14), U3.11 (SRCLK)
- new net SR_DATA: U2.16 (IO13), U3.14 (SER)
- new net SR_LATCH: U2.23 (IO15), U3.12 (RCLK)
- no-connect marks 0 -> 8
Other:
- note added: "asdasdasd"
